File: Hardware/AFE.sch (KiCad schematic (older format))
At the start: 0 parts

Commit message: Getting down structure, some components created.
Parts:
- added C1: 220pF, GaudiLabsFootPrints:0805G, symbol OpenThereminCC-rescue:C
- added C10, C2, C3, C9: 150pF, GaudiLabsFootPrints:0805G, symbol OpenThereminCC-rescue:C
- added C11: 10pF, GaudiLabsFootPrints:0805G, symbol OpenThereminCC-rescue:C
- added C12, C5: 470pF, GaudiLabsFootPrints:0805G, symbol OpenThereminCC-rescue:C
- added C13, C23, C24, C25, C26, C27, C28, C6: 100nF, GaudiLabsFootPrints:0805G, symbol OpenThereminCC-rescue:C
- added C14, C4, C7: not assembled, GaudiLabsFootPrints:0805G, symbol OpenThereminCC-rescue:C
- added C20: 100n, GaudiLabsFootPrints:0805G, symbol OpenThereminCC-rescue:C
- added C8: 330pF, GaudiLabsFootPrints:0805G, symbol OpenThereminCC-rescue:C
- added D1, D2: BB914, TO_SOT_Packages_SMD:SOT-23, symbol OpenThereminCC-rescue:CapDiode
- added GROUND1: GND_PAD, GaudiLabsFootPrints:MountPad3, symbol OpenThereminCC-rescue:TEST_1P
- added L1, L2: 1mH, GaudiLabsFootPrints:COIL, symbol OpenThereminCC-rescue:FILTER
- added R1, R5: 4.7M, GaudiLabsFootPrints:0805G, symbol OpenThereminCC-rescue:RES
- added R15, R3, R4, R7, R8: 100k, GaudiLabsFootPrints:0805G, symbol OpenThereminCC-rescue:RES
- added R2, R6: 2.2k, GaudiLabsFootPrints:0805G, symbol OpenThereminCC-rescue:RES
- added TP801: VO_PITCH, TestPoint:TestPoint_THTPad_D1.5mm_Drill0.7mm, symbol Connector:TestPoint
- added TP802: VO_VOL, TestPoint:TestPoint_THTPad_D1.5mm_Drill0.7mm, symbol Connector:TestPoint
- added U5: 4069, GaudiLabsFootPrints:SOIC-14_N, symbol OpenThereminCC-rescue:4069
- added U801: MCP47CXBX2, Package_DFN_QFN:DFN-10-1EP_3x3mm_P0.5mm_EP1.55x2.48mm, symbol OHMC2022:MCP47CXBX2
- added W1: FIDUCIAL1, Fiducials:Fiducial_1mm_Dia_2.54mm_Outer_CopperTop, symbol OpenThereminCC-rescue:TEST_1P
- added W2: FIDUCIAL2, Fiducials:Fiducial_1mm_Dia_2.54mm_Outer_CopperTop, symbol OpenThereminCC-rescue:TEST_1P
- added Y1, Y2: MountPad3, GaudiLabsFootPrints:MountPad3, symbol OpenThereminCC-rescue:MountPad3
Connections:
- net labels added: DAC_LATCH, GND, VCC, VDD, VO_PITCH, VO_VOL, VSS, VoutA, VoutB, VrefB
- wire segments 0 -> 125
Other:
- note added: "220pF?\n"
- note added: "Change DAC to i2c"
- note added: "Level convert if using +5V"
- note added: "TEST POINTS!!"
