File: Hardware/Amplifier.sch (KiCad schematic (older format))
At the start: 12 parts, among them U401 PAM8019KGR

Commit message: Commit before branch to fix VIN=3v3 from SAO.
Connections:
- net GND: now also U401.10 (HP/~SPK)
Changed lines of the file:
@@
 	3650 2250 4350 2250
 Connection ~ 4350 2250
+$Comp
+L power:GND #PWR?
+U 1 1 6140FAB1
+P 4650 4900
+AR Path="/611E3335/6140FAB1" Ref="#PWR?"  Part="1"
+AR Path="/611E3218/611E330D/6140FAB1" Ref="#PWR?"  Part="1"
+F 0 "#PWR?" H 4650 4650 50  0001 C CNN
+F 1 "GND" H 4655 4727 50  0000 C CNN
+F 2 "" H 4650 4900 50  0001 C CNN
+F 3 "" H 4650 4900 50  0001 C CNN
+	1    4650 4900
+	-1   0    0    -1
+$EndComp
+Wire Wire Line
+	4750 4650 4650 4650
+Wire Wire Line
+	4650 4650 4650 4900
 $EndSCHEMATC

Commit message: Fixing up some BoM repetition.
Parts:
- R401, R402: footprint Resistor_SMD:R_0603_1608Metric -> Resistor_SMD:R_0402_1005Metric
Changed lines of the file:
@@
 F 0 "R402" H 6870 4196 50  0000 L CNN
 F 1 "DNF" H 6870 4105 50  0000 L CNN
-F 2 "Resistor_SMD:R_0603_1608Metric" V 6730 4150 50  0001 C CNN
+F 2 "Resistor_SMD:R_0402_1005Metric" V 6730 4150 50  0001 C CNN
 F 3 "~" H 6800 4150 50  0001 C CNN
 	1    6800 4150
@@
 F 0 "R401" H 6870 3646 50  0000 L CNN
 F 1 "DNF" H 6870 3555 50  0000 L CNN
-F 2 "Resistor_SMD:R_0603_1608Metric" V 6730 3600 50  0001 C CNN
+F 2 "Resistor_SMD:R_0402_1005Metric" V 6730 3600 50  0001 C CNN
 F 3 "~" H 6800 3600 50  0001 C CNN
 	1    6800 3600

Commit message: Trying to add suppliers in Altium formats.
Parts:
- C403: Supplier 1 (none) -> Digi-Key; Supplier Part Number 1 (none) -> 399-6856-1-ND
- C404, C405: Supplier 1 (none) -> Digi-Key; Supplier Part Number 1 (none) -> 587-3352-1-ND
- R405: Supplier 1 (none) -> Digi-Key; Supplier Part Number 1 (none) -> RNCP0603FTD10K0CT-ND
- U401: MouserPN 621-PAM8019KGR -> 621-PAM8019KGR; Supplier 1 (none) -> Mouser; Supplier Part Number 1 (none) -> 621-PAM8019KGR
- U401: MPN (none) -> PAM8019KGR; MouserPN (none) -> 621-PAM8019KGR; Supplier 1 (none) -> Mouser; Supplier Part Number 1 (none) -> 621-PAM8019KGR
Changed lines of the file:
@@
 F 3 "www.diodes.com/assets/Datasheets/PAM8019.pdf" H 5100 2850 50  0001 C CNN
 F 4 "PAM8019KGR" H 5400 3850 50  0001 C CNN "MPN"
-F 5 "621-PAM8019KGR " H 5400 3850 50  0001 C CNN "MouserPN"
+F 5 "621-PAM8019KGR" H 5400 3850 50  0001 C CNN "MouserPN"
+F 6 "Mouser" H 5400 3850 50  0001 C CNN "Supplier 1"
+F 7 "621-PAM8019KGR" H 5400 3850 50  0001 C CNN "Supplier Part Number 1"
 	1    5400 3850
 	1    0    0    -1
@@
 F 2 "Package_DFN_QFN:QFN-20-1EP_4x4mm_P0.5mm_EP2.6x2.6mm" H 4750 900 50  0001 C CNN
 F 3 "www.diodes.com/assets/Datasheets/PAM8019.pdf" H 4750 900 50  0001 C CNN
+F 4 "PAM8019KGR" H 5050 1900 50  0001 C CNN "MPN"
+F 5 "621-PAM8019KGR" H 5050 1900 50  0001 C CNN "MouserPN"
+F 6 "Mouser" H 5050 1900 50  0001 C CNN "Supplier 1"
+F 7 "621-PAM8019KGR" H 5050 1900 50  0001 C CNN "Supplier Part Number 1"
 	2    5050 1900
 	1    0    0    -1
@@
 F 7 "0603" H 3965 4559 50  0000 L CNN "Pkg"
 F 8 "X7R" H 3965 4468 50  0000 L CNN "TCoff"
+F 9 "Digi-Key" H 3850 4650 50  0001 C CNN "Supplier 1"
+F 10 "587-3352-1-ND" H 3850 4650 50  0001 C CNN "Supplier Part Number 1"
 	1    3850 4650
 	1    0    0    -1
@@
 F 7 "0603" H 4465 1909 50  0000 L CNN "Pkg"
 F 8 "X7R" H 4465 1818 50  0000 L CNN "TCoff"
+F 9 "Digi-Key" H 4350 2000 50  0001 C CNN "Supplier 1"
+F 10 "587-3352-1-ND" H 4350 2000 50  0001 C CNN "Supplier Part Number 1"
 	1    4350 2000
 	-1   0    0    -1
@@
 F 5 "RNCP0603FTD10K0" H 3050 4650 50  0001 C CNN "MPN"
 F 6 "RNCP0603FTD10K0CT-ND" H 3050 4650 50  0001 C CNN "DPN"
+F 7 "Digi-Key" H 3050 4650 50  0001 C CNN "Supplier 1"
+F 8 "RNCP0603FTD10K0CT-ND" H 3050 4650 50  0001 C CNN "Supplier Part Number 1"
 	1    3050 4650
 	1    0    0    -1
@@
 F 7 "0603" H 3765 1909 50  0000 L CNN "Pkg"
 F 8 "X7R" H 3765 1818 50  0000 L CNN "TCoff"
+F 9 "Digi-Key" H 3650 2000 50  0001 C CNN "Supplier 1"
+F 10 "399-6856-1-ND" H 3650 2000 50  0001 C CNN "Supplier Part Number 1"
 	1    3650 2000
 	1    0    0    -1
