File: Hardware/Codec.sch (KiCad schematic (older format))
At the start: 0 parts

Commit message: Getting down structure, some components created.
Parts:
- added U301: SGTL5000XNAA3, Package_DFN_QFN:QFN-32-1EP_5x5mm_P0.5mm_EP3.65x3.65mm_ThermalVias, symbol SGTL5000XNAA:SGTL5000XNAA3
Changed lines of the file:
@@
 Comment4 ""
 $EndDescr
+$Comp
+L SGTL5000XNAA:SGTL5000XNAA3 U301
+U 1 1 61232CBC
+P 5250 3450
+AR Path="/611E3218/611E32E1/61232CBC" Ref="U301"  Part="1"
+AR Path="/61375092/611E32E1/61232CBC" Ref="U?"  Part="1"
+F 0 "U301" H 5250 4817 50  0000 C CNN
+F 1 "SGTL5000XNAA3" H 5250 4726 50  0000 C CNN
+F 2 "Package_DFN_QFN:QFN-32-1EP_5x5mm_P0.5mm_EP3.65x3.65mm_ThermalVias" H 5250 3450 50  0001 L BNN
+F 3 "" H 5250 3450 50  0001 L BNN
+F 4 "Freescale Semiconductor" H 5250 3450 50  0001 L BNN "MANUFACTURER"
+	1    5250 3450
+	1    0    0    -1
+$EndComp
+Text HLabel 7100 2850 2    50   Output ~ 0
+LineOut_R
+Text HLabel 7100 2950 2    50   Output ~ 0
+LineOut_L
 $EndSCHEMATC
