File: Hardware/Codec.sch (KiCad schematic (older format))
At the start: 14 parts, among them U301 SGTL5000XNAA3

Commit message: Trying to add suppliers in Altium formats.
Parts:
- C301, C305, C307, C606: Supplier 1 (none) -> Digi-Key; Supplier Part Number 1 (none) -> 399-6856-1-ND
- C302, C304, C308, C309, C608, C611: Supplier 1 (none) -> Digi-Key; Supplier Part Number 1 (none) -> 587-3352-1-ND
- FB601: Supplier 1 (none) -> Digi-Key; Supplier Part Number 1 (none) -> 490-1014-1-ND
- U301: Supplier 1 (none) -> Digi-Key; Supplier Part Number 1 (none) -> SGTL5000XNAA3-ND
Changed lines of the file:
@@
 F 7 "0603" H 3515 1859 50  0000 L CNN "Pkg"
 F 8 "X7R" H 3515 1768 50  0000 L CNN "TCoff"
+F 9 "Digi-Key" H 3400 1950 50  0001 C CNN "Supplier 1"
+F 10 "587-3352-1-ND" H 3400 1950 50  0001 C CNN "Supplier Part Number 1"
 	1    3400 1950
 	1    0    0    -1
@@
 F 7 "0603" H 4015 1859 50  0000 L CNN "Pkg"
 F 8 "X7R" H 4015 1768 50  0000 L CNN "TCoff"
+F 9 "Digi-Key" H 3900 1950 50  0001 C CNN "Supplier 1"
+F 10 "399-6856-1-ND" H 3900 1950 50  0001 C CNN "Supplier Part Number 1"
 	1    3900 1950
 	1    0    0    -1
@@
 F 7 "0603" H 2215 3059 50  0000 L CNN "Pkg"
 F 8 "X7R" H 2215 2968 50  0000 L CNN "TCoff"
+F 9 "Digi-Key" H 2100 3150 50  0001 C CNN "Supplier 1"
+F 10 "399-6856-1-ND" H 2100 3150 50  0001 C CNN "Supplier Part Number 1"
 	1    2100 3150
 	0    1    1    0
@@
 F 5 "SGTL5000XNAA3" H 5250 3450 50  0001 C CNN "MPN"
 F 6 "SGTL5000XNAA3-ND" H 5250 3450 50  0001 C CNN "DPN"
+F 7 "Digi-Key" H 5250 3450 50  0001 C CNN "Supplier 1"
+F 8 "SGTL5000XNAA3-ND" H 5250 3450 50  0001 C CNN "Supplier Part Number 1"
 	1    5250 3450
 	1    0    0    -1
@@
 F 7 "0603" H 6815 4009 50  0000 L CNN "Pkg"
 F 8 "X7R" H 6815 3918 50  0000 L CNN "TCoff"
+F 9 "Digi-Key" H 6700 4100 50  0001 C CNN "Supplier 1"
+F 10 "399-6856-1-ND" H 6700 4100 50  0001 C CNN "Supplier Part Number 1"
 	1    6700 4100
 	1    0    0    -1
@@
 F 7 "0603" H 2915 3509 50  0000 L CNN "Pkg"
 F 8 "X7R" H 2915 3418 50  0000 L CNN "TCoff"
+F 9 "Digi-Key" H 2800 3600 50  0001 C CNN "Supplier 1"
+F 10 "587-3352-1-ND" H 2800 3600 50  0001 C CNN "Supplier Part Number 1"
 	1    2800 3600
 	1    0    0    -1
@@
 F 7 "0603" H 7365 2759 50  0000 L CNN "Pkg"
 F 8 "X7R" H 7365 2668 50  0000 L CNN "TCoff"
+F 9 "Digi-Key" H 7250 2850 50  0001 C CNN "Supplier 1"
+F 10 "587-3352-1-ND" H 7250 2850 50  0001 C CNN "Supplier Part Number 1"
 	1    7250 2850
 	0    -1   -1   0
@@
 F 7 "0603" H 6965 2859 50  0000 L CNN "Pkg"
 F 8 "X7R" H 6965 2768 50  0000 L CNN "TCoff"
+F 9 "Digi-Key" H 6850 2950 50  0001 C CNN "Supplier 1"
+F 10 "587-3352-1-ND" H 6850 2950 50  0001 C CNN "Supplier Part Number 1"
 	1    6850 2950
 	0    -1   1    0
@@
 F 4 "BLM18AG601SN1D" V 5250 1650 50  0001 C CNN "MPN"
 F 5 "490-1014-1-ND" V 5250 1650 50  0001 C CNN "DPN"
+F 6 "Digi-Key" H 5250 1650 50  0001 C CNN "Supplier 1"
+F 7 "490-1014-1-ND" H 5250 1650 50  0001 C CNN "Supplier Part Number 1"
 	1    5250 1650
 	0    1    1    0
@@
 F 7 "0603" H 7265 1909 50  0000 L CNN "Pkg"
 F 8 "X7R" H 7265 1818 50  0000 L CNN "TCoff"
+F 9 "Digi-Key" H 7150 2000 50  0001 C CNN "Supplier 1"
+F 10 "587-3352-1-ND" H 7150 2000 50  0001 C CNN "Supplier Part Number 1"
 	1    7150 2000
 	1    0    0    1
@@
 F 7 "0603" H 6815 1909 50  0000 L CNN "Pkg"
 F 8 "X7R" H 6815 1818 50  0000 L CNN "TCoff"
+F 9 "Digi-Key" H 6700 2000 50  0001 C CNN "Supplier 1"
+F 10 "587-3352-1-ND" H 6700 2000 50  0001 C CNN "Supplier Part Number 1"
 	1    6700 2000
 	1    0    0    -1
@@
 F 7 "0603" H 6515 1909 50  0000 L CNN "Pkg"
 F 8 "X7R" H 6515 1818 50  0000 L CNN "TCoff"
+F 9 "Digi-Key" H 6400 2000 50  0001 C CNN "Supplier 1"
+F 10 "399-6856-1-ND" H 6400 2000 50  0001 C CNN "Supplier Part Number 1"
 	1    6400 2000
 	-1   0    0    1

Commit message: Cleaning up some libraries, better if those pins are connected.
Changed lines of the file:
@@
 Wire Wire Line
 	3400 2100 3400 2550
+$Comp
+L power:PWR_FLAG #FLG?
+U 1 1 61817384
+P 7150 1500
+AR Path="/61817384" Ref="#FLG?"  Part="1"
+AR Path="/611E335F/61817384" Ref="#FLG?"  Part="1"
+AR Path="/611E3218/611E32E1/61817384" Ref="#FLG0109"  Part="1"
+F 0 "#FLG0109" H 7150 1575 50  0001 C CNN
+F 1 "PWR_FLAG" H 7150 1673 50  0000 C CNN
+F 2 "" H 7150 1500 50  0001 C CNN
+F 3 "~" H 7150 1500 50  0001 C CNN
+	1    7150 1500
+	1    0    0    -1
+$EndComp
+Wire Wire Line
+	7150 1500 7150 1650
+Connection ~ 7150 1650
 $EndSCHEMATC

Commit message: Changing around the audio inputs.
Connections:
- net LINE_IN_R: now reaches U301.13 (LINEIN_R)
- no-connect marks 3 -> 2
Changed lines of the file:
@@
  Do not connect HP_VGND to system ground, even\nwhen unused. This is a virtual ground (DC voltage) that\nshould never connect to an actual “0 Volt ground”. Use\nthe widest, shortest trace possible for the HP_VGND.\n
 NoConn ~ 6050 3950
-NoConn ~ 4450 2850
 NoConn ~ 4450 2950
 $Comp
@@
 	7150 1500 7150 1650
 Connection ~ 7150 1650
+Text HLabel 1850 2850 0    50   Input ~ 0
+LINE_IN_R
+Wire Wire Line
+	4450 2850 1850 2850
 $EndSCHEMATC

Commit message: Adding resistor to line-in just in case.
Parts:
- added R?: 22R, Resistor_SMD:R_0603_1608Metric, symbol Device:R
Connections:
- net LINE_IN_R: now also R?.2; no longer U301.13 (LINEIN_R)
- new net: R?.1, U301.13 (LINEIN_R)
Changed lines of the file:
@@
 Text HLabel 1850 2850 0    50   Input ~ 0
 LINE_IN_R
+$Comp
+L Device:R R?
+U 1 1 61421EF9
+P 2600 2850
+AR Path="/61421EF9" Ref="R?"  Part="1"
+AR Path="/611E3335/61421EF9" Ref="R?"  Part="1"
+AR Path="/611E3218/611E32E1/61421EF9" Ref="R?"  Part="1"
+F 0 "R?" V 2393 2850 50  0000 C CNN
+F 1 "22R" V 2484 2850 50  0000 C CNN
+F 2 "Resistor_SMD:R_0603_1608Metric" V 2530 2850 50  0001 C CNN
+F 3 "~" H 2600 2850 50  0001 C CNN
+F 4 "CRGCQ0603J22R" V 2600 2850 50  0001 C CNN "MPN"
+F 5 "A130081CT-ND" V 2600 2850 50  0001 C CNN "DPN"
+F 6 "Digi-Key" H 2600 2850 50  0001 C CNN "Supplier 1"
+F 7 "A130081CT-ND" H 2600 2850 50  0001 C CNN "Supplier Part Number 1"
+	1    2600 2850
+	0    1    1    0
+$EndComp
 Wire Wire Line
-	4450 2850 1850 2850
+	1850 2850 2450 2850
+Wire Wire Line
+	2750 2850 4450 2850
 $EndSCHEMATC

Commit message: Going to regenerate BoM.
Parts:
- gave numbers to parts that had none: 1
Changed lines of the file:
@@
 AR Path="/61421EF9" Ref="R?"  Part="1"
 AR Path="/611E3335/61421EF9" Ref="R?"  Part="1"
-AR Path="/611E3218/611E32E1/61421EF9" Ref="R?"  Part="1"
-F 0 "R?" V 2393 2850 50  0000 C CNN
+AR Path="/611E3218/611E32E1/61421EF9" Ref="R602"  Part="1"
+F 0 "R602" V 2393 2850 50  0000 C CNN
 F 1 "22R" V 2484 2850 50  0000 C CNN
 F 2 "Resistor_SMD:R_0603_1608Metric" V 2530 2850 50  0001 C CNN
