File: Hardware/Connectors.sch (KiCad schematic (older format))
At the start: 0 parts

Commit message: Getting down structure, some components created.
Parts:
- added J701: SpeakerOut, Connector_JST:JST_PH_S4B-PH-K_1x04_P2.00mm_Horizontal, symbol Connector:Conn_01x04_Male
- added J702: Conn_02x03_Odd_Even, RocklingLib:SAO_Header_6-Pin, symbol Connector_Generic:Conn_02x03_Odd_Even
Changed lines of the file:
@@
 $Descr A4 11693 8268
 encoding utf-8
-Sheet 1 8
+Sheet 7 8
 Title ""
 Date ""
@@
 Comment4 ""
 $EndDescr
+$Comp
+L Connector:Conn_01x04_Male J701
+U 1 1 6122FCF1
+P 8100 2400
+F 0 "J701" H 8208 2681 50  0000 C CNN
+F 1 "SpeakerOut" H 8208 2590 50  0000 C CNN
+F 2 "Connector_JST:JST_PH_S4B-PH-K_1x04_P2.00mm_Horizontal" H 8100 2400 50  0001 C CNN
+F 3 "~" H 8100 2400 50  0001 C CNN
+	1    8100 2400
+	1    0    0    -1
+$EndComp
+$Comp
+L Connector_Generic:Conn_02x03_Odd_Even J702
+U 1 1 612309ED
+P 8250 3800
+F 0 "J702" H 8300 4117 50  0000 C CNN
+F 1 "Conn_02x03_Odd_Even" H 8300 4026 50  0000 C CNN
+F 2 "RocklingLib:SAO_Header_6-Pin" H 8250 3800 50  0001 C CNN
+F 3 "~" H 8250 3800 50  0001 C CNN
+	1    8250 3800
+	1    0    0    -1
+$EndComp
 $EndSCHEMATC
