File: Hardware/Power.sch (KiCad schematic (older format))
At the start: 0 parts

Commit message: Getting down structure, some components created.
Parts:
- added C601, C602, C603, C604, C605, C606: 0201, 1uF, 10V, X5R, 20%, tomu-fpga:C_0201_0603Metric, symbol Device:C_Small
- added U601, U602: PAM2306AYPAA, Package_DFN_QFN:WDFN-12-1EP_3x3mm_P0.45mm_EP1.7x2.5mm, symbol Regulator_Switching:PAM2306AYPAA
- added U603: LDO-X2SON-1.2V, tomu-fpga:Texas_X2SON-4_1x1mm_P0.65mm, symbol tomu-fpga:LDO-X2SON
- added U604: LDO-X2SON-3.3V, tomu-fpga:Texas_X2SON-4_1x1mm_P0.65mm, symbol tomu-fpga:LDO-X2SON
- added U605: LDO-X2SON-2.5V, tomu-fpga:Texas_X2SON-4_1x1mm_P0.65mm, symbol tomu-fpga:LDO-X2SON
Connections:
- new net: U602.13 (GND), U602.3 (GND), U602.9 (GND)
- new net: U601.13 (GND), U601.3 (GND), U601.9 (GND)
- new net +1V2: C604.1, U603.1 (OUT), U604.3 (EN)
- new net +2V5: C606.1, U605.1 (OUT)
- new net +3V3: C605.1, U604.1 (OUT), U605.3 (EN)
- new net +5V: C601.1, C602.1, C603.1, U603.3 (EN), U603.4 (IN), U604.4 (IN), U605.4 (IN)
- new net GND: C601.2, C602.2, C603.2, C604.2, C605.2, C606.2, U603.2 (GND), U603.5 (Thermal), U604.2 (GND), U604.5 (Thermal), U605.2 (GND), U605.5 (Thermal)
Other:
- note added: "PCB Power Regulation"
- note added: "Power sequencing:\n1) 1.2V (VCC/VCCPLL)\n2) 3.3V (SPI_VCCIO1)\n3) 2.5V (VPP_2V5)\nSubsequent rails activate\nafter previous rail goes >0.5V"
