File: Hardware/Power.sch (KiCad schematic (older format))
At the start: 24 parts, among them U601 PAM2306AYPAA, U602 MIC5317-2.5YM5, U603 SiP32431DR3

Commit message: Fixing up some BoM repetition.
Other:
- moved on the sheet: C607, C610, R601, R610, U603
Changed lines of the file:
@@
 L Device:C C610
 U 1 1 612D6875
-P 9900 1400
-F 0 "C610" H 10015 1537 50  0000 L CNN
-F 1 "10uF" H 10015 1446 50  0000 L CNN
-F 2 "Capacitor_SMD:C_0603_1608Metric" H 9938 1250 50  0001 C CNN
-F 3 "~" H 9900 1400 50  0001 C CNN
-F 4 "GRM188R60J106ME47D" H 9900 1400 50  0001 C CNN "MPN"
-F 5 "490-3896-1-ND" H 9900 1400 50  0001 C CNN "DPN"
-F 6 "6.3V" H 10015 1355 50  0000 L CNN "Tol"
-F 7 "0603" H 10015 1264 50  0000 L CNN "Pkg"
-	1    9900 1400
+P 7950 1500
+F 0 "C610" H 8065 1637 50  0000 L CNN
+F 1 "10uF" H 8065 1546 50  0000 L CNN
+F 2 "Capacitor_SMD:C_0603_1608Metric" H 7988 1350 50  0001 C CNN
+F 3 "~" H 7950 1500 50  0001 C CNN
+F 4 "GRM188R60J106ME47D" H 7950 1500 50  0001 C CNN "MPN"
+F 5 "490-3896-1-ND" H 7950 1500 50  0001 C CNN "DPN"
+F 6 "6.3V" H 8065 1455 50  0000 L CNN "Tol"
+F 7 "0603" H 8065 1364 50  0000 L CNN "Pkg"
+	1    7950 1500
 	1    0    0    -1
 $EndComp
@@
 L power:+3V3 #PWR?
 U 1 1 613CFE20
-P 9900 1200
+P 7950 1300
 AR Path="/6123BB15/613CFE20" Ref="#PWR?"  Part="1"
 AR Path="/611E335F/613CFE20" Ref="#PWR0116"  Part="1"
-F 0 "#PWR0116" H 9900 1050 50  0001 C CNN
-F 1 "+3V3" H 9915 1373 50  0000 C CNN
-F 2 "" H 9900 1200 50  0001 C CNN
-F 3 "" H 9900 1200 50  0001 C CNN
-	1    9900 1200
+F 0 "#PWR0116" H 7950 1150 50  0001 C CNN
+F 1 "+3V3" H 7965 1473 50  0000 C CNN
+F 2 "" H 7950 1300 50  0001 C CNN
+F 3 "" H 7950 1300 50  0001 C CNN
+	1    7950 1300
 	1    0    0    -1
 $EndComp
@@
 L power:GND #PWR?
 U 1 1 613D467C
-P 9900 1650
+P 7950 1750
 AR Path="/611E3335/613D467C" Ref="#PWR?"  Part="1"
 AR Path="/611E335F/613D467C" Ref="#PWR0118"  Part="1"
-F 0 "#PWR0118" H 9900 1400 50  0001 C CNN
-F 1 "GND" H 9905 1477 50  0000 C CNN
-F 2 "" H 9900 1650 50  0001 C CNN
-F 3 "" H 9900 1650 50  0001 C CNN
-	1    9900 1650
-	-1   0    0    -1
-$EndComp
-Wire Wire Line
-	9900 1550 9900 1650
+F 0 "#PWR0118" H 7950 1500 50  0001 C CNN
+F 1 "GND" H 7955 1577 50  0000 C CNN
+F 2 "" H 7950 1750 50  0001 C CNN
+F 3 "" H 7950 1750 50  0001 C CNN
+	1    7950 1750
+	-1   0    0    -1
+$EndComp
+Wire Wire Line
+	7950 1650 7950 1750
 Wire Wire Line
 	6350 3850 6350 3950
@@
 	6350 3500 6350 3550
 Wire Wire Line
-	9900 1200 9900 1250
+	7950 1300 7950 1350
 Wire Wire Line
 	2500 3550 2600 3550
@@
 L power:+3V3 #PWR?
 U 1 1 613C426F
-P 9500 1200
+P 7550 1300
 AR Path="/6123BB15/613C426F" Ref="#PWR?"  Part="1"
 AR Path="/611E335F/613C426F" Ref="#PWR0113"  Part="1"
-F 0 "#PWR0113" H 9500 1050 50  0001 C CNN
-F 1 "+3V3" H 9515 1373 50  0000 C CNN
-F 2 "" H 9500 1200 50  0001 C CNN
-F 3 "" H 9500 1200 50  0001 C CNN
-	1    9500 1200
+F 0 "#PWR0113" H 7550 1150 50  0001 C CNN
+F 1 "+3V3" H 7565 1473 50  0000 C CNN
+F 2 "" H 7550 1300 50  0001 C CNN
+F 3 "" H 7550 1300 50  0001 C CNN
+	1    7550 1300
 	1    0    0    -1
 $EndComp
@@
 L Device:R_Small_US R601
 U 1 1 612EE9BF
-P 7750 1550
-F 0 "R601" H 7818 1596 50  0000 L CNN
-F 1 "100K" H 7818 1505 50  0000 L CNN
-F 2 "Resistor_SMD:R_0603_1608Metric" V 7680 1550 50  0001 C CNN
-F 3 "~" H 7750 1550 50  0001 C CNN
-F 4 "0603" H 7750 1550 50  0001 C CNN "Pkg"
-F 5 "ESR03EZPJ104" H 7750 1550 50  0001 C CNN "MPN"
-F 6 "RHM100KDCT-ND" H 7750 1550 50  0001 C CNN "DPN"
-	1    7750 1550
+P 5800 1650
+F 0 "R601" H 5868 1696 50  0000 L CNN
+F 1 "100K" H 5868 1605 50  0000 L CNN
+F 2 "Resistor_SMD:R_0603_1608Metric" V 5730 1650 50  0001 C CNN
+F 3 "~" H 5800 1650 50  0001 C CNN
+F 4 "0603" H 5800 1650 50  0001 C CNN "Pkg"
+F 5 "ESR03EZPJ104" H 5800 1650 50  0001 C CNN "MPN"
+F 6 "RHM100KDCT-ND" H 5800 1650 50  0001 C CNN "DPN"
+	1    5800 1650
 	1    0    0    -1
 $EndComp
@@
 	2600 3550 3650 3550
 Wire Wire Line
-	7750 1350 7750 1450
+	5800 1450 5800 1550
 Wire Wire Line
 	3650 3950 3300 3950
@@
 L Power_Management:SiP32431DR3 U603
 U 1 1 615CC64C
-P 9050 1800
-F 0 "U603" H 9050 2167 50  0000 C CNN
-F 1 "SiP32431DR3" H 9050 2076 50  0000 C CNN
-F 2 "Package_TO_SOT_SMD:SOT-363_SC-70-6" H 9050 2250 50  0001 C CNN
-F 3 "https://www.vishay.com/docs/66597/sip32431.pdf" H 9050 1800 50  0001 C CNN
-F 4 "SIP32431DR3-T1GE3" H 9050 1800 50  0001 C CNN "MPN"
-F 5 "SIP32431DR3-T1GE3CT-ND" H 9050 1800 50  0001 C CNN "DPN"
-	1    9050 1800
-	1    0    0    -1
-$EndComp
-Wire Wire Line
-	8300 1800 8750 1800
-Connection ~ 8300 1800
-Connection ~ 7750 1800
-Wire Wire Line
-	7750 1800 8300 1800
-Wire Wire Line
-	7750 1650 7750 1800
+P 7100 1900
+F 0 "U603" H 7100 2267 50  0000 C CNN
+F 1 "SiP32431DR3" H 7100 2176 50  0000 C CNN
+F 2 "Package_TO_SOT_SMD:SOT-363_SC-70-6" H 7100 2350 50  0001 C CNN
+F 3 "https://www.vishay.com/docs/66597/sip32431.pdf" H 7100 1900 50  0001 C CNN
+F 4 "SIP32431DR3-T1GE3" H 7100 1900 50  0001 C CNN "MPN"
+F 5 "SIP32431DR3-T1GE3CT-ND" H 7100 1900 50  0001 C CNN "DPN"
+	1    7100 1900
+	1    0    0    -1
+$EndComp
+Wire Wire Line
+	6350 1900 6800 1900
+Connection ~ 6350 1900
+Connection ~ 5800 1900
+Wire Wire Line
+	5800 1900 6350 1900
+Wire Wire Line
+	5800 1750 5800 1900
 $Comp
 L Device:C C607
 U 1 1 612DE99A
-P 7750 2150
-F 0 "C607" H 7865 2332 50  0000 L CNN
-F 1 "1uF" H 7865 2241 50  0000 L CNN
-F 2 "Capacitor_SMD:C_0603_1608Metric" H 7788 2000 50  0001 C CNN
-F 3 "~" H 7750 2150 50  0001 C CNN
-F 4 "GMK107AB7105KAHT" H 7750 2150 50  0001 C CNN "MPN"
-F 5 "587-3352-1-ND" H 7750 2150 50  0001 C CNN "DPN"
-F 6 "35V" H 7865 2150 50  0000 L CNN "Tol"
-F 7 "0603" H 7865 2059 50  0000 L CNN "Pkg"
-F 8 "X7R" H 7865 1968 50  0000 L CNN "TCoff"
-	1    7750 2150
+P 5800 2250
+F 0 "C607" H 5915 2432 50  0000 L CNN
+F 1 "1uF" H 5915 2341 50  0000 L CNN
+F 2 "Capacitor_SMD:C_0603_1608Metric" H 5838 2100 50  0001 C CNN
+F 3 "~" H 5800 2250 50  0001 C CNN
+F 4 "GMK107AB7105KAHT" H 5800 2250 50  0001 C CNN "MPN"
+F 5 "587-3352-1-ND" H 5800 2250 50  0001 C CNN "DPN"
+F 6 "35V" H 5915 2250 50  0000 L CNN "Tol"
+F 7 "0603" H 5915 2159 50  0000 L CNN "Pkg"
+F 8 "X7R" H 5915 2068 50  0000 L CNN "TCoff"
+	1    5800 2250
 	1    0    0    -1
 $EndComp
@@
 L Device:R_Small R610
 U 1 1 61513F81
-P 8300 2200
+P 6350 2300
 AR Path="/611E335F/61513F81" Ref="R610"  Part="1"
 AR Path="/61513F81" Ref="R?"  Part="1"
-F 0 "R610" H 8350 2250 50  0000 L CNN
-F 1 "1M" H 8350 2150 50  0000 L CNN
-F 2 "Resistor_SMD:R_0603_1608Metric" V 8230 2200 50  0001 C CNN
-F 3 "~" H 8300 2200 50  0001 C CNN
-F 4 "0603" H 8450 2350 50  0000 C CNN "Pkg"
-F 5 "CR0603-JW-105ELF" H 8300 2200 50  0001 C CNN "MPN"
-F 6 "CR0603-JW-105ELFCT-ND" H 8300 2200 50  0001 C CNN "DPN"
-	1    8300 2200
-	1    0    0    -1
-$EndComp
-Wire Wire Line
-	8300 1800 8300 2100
-Wire Wire Line
-	8300 2300 8300 2650
+F 0 "R610" H 6400 2350 50  0000 L CNN
+F 1 "1M" H 6400 2250 50  0000 L CNN
+F 2 "Resistor_SMD:R_0603_1608Metric" V 6280 2300 50  0001 C CNN
+F 3 "~" H 6350 2300 50  0001 C CNN
+F 4 "0603" H 6500 2450 50  0000 C CNN "Pkg"
+F 5 "CR0603-JW-105ELF" H 6350 2300 50  0001 C CNN "MPN"
+F 6 "CR0603-JW-105ELFCT-ND" H 6350 2300 50  0001 C CNN "DPN"
+	1    6350 2300
+	1    0    0    -1
+$EndComp
+Wire Wire Line
+	6350 1900 6350 2200
+Wire Wire Line
+	6350 2400 6350 2750
 $Comp
 L power:GND #PWR?
 U 1 1 6151831E
-P 8300 2650
+P 6350 2750
 AR Path="/611E3335/6151831E" Ref="#PWR?"  Part="1"
 AR Path="/611E335F/6151831E" Ref="#PWR0135"  Part="1"
-F 0 "#PWR0135" H 8300 2400 50  0001 C CNN
-F 1 "GND" H 8305 2477 50  0000 C CNN
-F 2 "" H 8300 2650 50  0001 C CNN
-F 3 "" H 8300 2650 50  0001 C CNN
-	1    8300 2650
+F 0 "#PWR0135" H 6350 2500 50  0001 C CNN
+F 1 "GND" H 6355 2577 50  0000 C CNN
+F 2 "" H 6350 2750 50  0001 C CNN
+F 3 "" H 6350 2750 50  0001 C CNN
+	1    6350 2750
 	-1   0    0    -1
 $EndComp
@@
 L power:GND #PWR?
 U 1 1 613EC141
-P 7750 2650
+P 5800 2750
 AR Path="/611E3335/613EC141" Ref="#PWR?"  Part="1"
 AR Path="/611E335F/613EC141" Ref="#PWR0120"  Part="1"
-F 0 "#PWR0120" H 7750 2400 50  0001 C CNN
-F 1 "GND" H 7755 2477 50  0000 C CNN
-F 2 "" H 7750 2650 50  0001 C CNN
-F 3 "" H 7750 2650 50  0001 C CNN
-	1    7750 2650
-	-1   0    0    -1
-$EndComp
-Wire Wire Line
-	7750 2650 7750 2300
-Wire Wire Line
-	7750 1800 7750 2000
-Wire Wire Line
-	8750 1700 8300 1700
-Wire Wire Line
-	8300 1700 8300 1350
-Wire Wire Line
-	8300 1350 7750 1350
-Wire Wire Line
-	9500 1200 9500 1700
-Wire Wire Line
-	9500 1700 9350 1700
+F 0 "#PWR0120" H 5800 2500 50  0001 C CNN
+F 1 "GND" H 5805 2577 50  0000 C CNN
+F 2 "" H 5800 2750 50  0001 C CNN
+F 3 "" H 5800 2750 50  0001 C CNN
+	1    5800 2750
+	-1   0    0    -1
+$EndComp
+Wire Wire Line
+	5800 2750 5800 2400
+Wire Wire Line
+	5800 1900 5800 2100
+Wire Wire Line
+	6800 1800 6350 1800
+Wire Wire Line
+	6350 1800 6350 1450
+Wire Wire Line
+	6350 1450 5800 1450
+Wire Wire Line
+	7550 1300 7550 1800
+Wire Wire Line
+	7550 1800 7400 1800
 Wire Wire Line
 	1900 3850 2200 3850
@@
 L power:VCCQ #PWR0133
 U 1 1 6163B616
-P 7750 1200
-F 0 "#PWR0133" H 7750 1050 50  0001 C CNN
-F 1 "VCCQ" H 7765 1373 50  0000 C CNN
-F 2 "" H 7750 1200 50  0001 C CNN
-F 3 "" H 7750 1200 50  0001 C CNN
-	1    7750 1200
+P 5800 1300
+F 0 "#PWR0133" H 5800 1150 50  0001 C CNN
+F 1 "VCCQ" H 5815 1473 50  0000 C CNN
+F 2 "" H 5800 1300 50  0001 C CNN
+F 3 "" H 5800 1300 50  0001 C CNN
+	1    5800 1300
 	1    0    0    -1
 $EndComp
@@
 	3300 3800 3300 3950
 Wire Wire Line
-	7750 1200 7750 1350
-Connection ~ 7750 1350
+	5800 1300 5800 1450
+Connection ~ 5800 1450
 Wire Wire Line
 	1550 3850 1900 3850
@@
 L power:GND #PWR?
 U 1 1 61660820
-P 9050 2650
+P 7100 2750
 AR Path="/611E3335/61660820" Ref="#PWR?"  Part="1"
 AR Path="/611E335F/61660820" Ref="#PWR0147"  Part="1"
-F 0 "#PWR0147" H 9050 2400 50  0001 C CNN
-F 1 "GND" H 9055 2477 50  0000 C CNN
-F 2 "" H 9050 2650 50  0001 C CNN
-F 3 "" H 9050 2650 50  0001 C CNN
-	1    9050 2650
-	-1   0    0    -1
-$EndComp
-Wire Wire Line
-	9050 2100 9050 2650
+F 0 "#PWR0147" H 7100 2500 50  0001 C CNN
+F 1 "GND" H 7105 2577 50  0000 C CNN
+F 2 "" H 7100 2750 50  0001 C CNN
+F 3 "" H 7100 2750 50  0001 C CNN
+	1    7100 2750
+	-1   0    0    -1
+$EndComp
+Wire Wire Line
+	7100 2200 7100 2750
 Wire Wire Line
 	1900 3200 1900 3550

Commit message: Backfeed enabled.
Parts:
- added JP?: Backfeed, OHMC2022:SolderJumper-2_P1.3mm_Open_RoundedPad1.0x1.5mm, symbol Device:Jumper_NO_Small
Connections:
- net +3V3: now also D602.3 (A2)
- net VIN: now also JP?.1
- net at D602.4 (K2): now also JP?.2
Other:
- note added: "Don't do this.\n(Do it. Do IT!)"
Changed lines of the file:
@@
 $Descr A4 11693 8268
 encoding utf-8
-Sheet 6 7
+Sheet 3 7
 Title ""
 Date ""
@@
 L power:VBUS #PWR?
 U 1 1 614E2688
-P 1300 2650
+P 1300 3200
 AR Path="/61291C71/614E2688" Ref="#PWR?"  Part="1"
 AR Path="/614E2688" Ref="#PWR?"  Part="1"
 AR Path="/611E335F/614E2688" Ref="#PWR0131"  Part="1"
-F 0 "#PWR0131" H 1300 2500 50  0001 C CNN
-F 1 "VBUS" H 1300 2800 50  0000 C CNN
-F 2 "" H 1300 2650 50  0001 C CNN
-F 3 "" H 1300 2650 50  0001 C CNN
-	1    1300 2650
+F 0 "#PWR0131" H 1300 3050 50  0001 C CNN
+F 1 "VBUS" H 1300 3350 50  0000 C CNN
+F 2 "" H 1300 3200 50  0001 C CNN
+F 3 "" H 1300 3200 50  0001 C CNN
+	1    1300 3200
 	1    0    0    -1
 $EndComp
@@
 	1350 3550 1300 3550
 Wire Wire Line
-	1300 3550 1300 2650
+	1300 3550 1300 3200
 $Comp
 L pkl_power:VIN #PWR0132
@@
 Wire Wire Line
 	3650 4400 3650 4750
+Wire Wire Line
+	650  4000 650  4150
+Wire Wire Line
+	650  4150 950  4150
+$Comp
+L pkl_power:VIN #PWR?
+U 1 1 61405D3E
+P 1550 4600
+F 0 "#PWR?" H 1550 4450 50  0001 C CNN
+F 1 "VIN" H 1550 4750 50  0000 C CNN
+F 2 "" H 1550 4600 50  0001 C CNN
+F 3 "" H 1550 4600 50  0001 C CNN
+	1    1550 4600
+	1    0    0    -1
+$EndComp
+$Comp
+L Device:Jumper_NO_Small JP?
+U 1 1 6141A32E
+P 1350 4600
+AR Path="/6141A32E" Ref="JP?"  Part="1"
+AR Path="/611E335F/6141A32E" Ref="JP?"  Part="1"
+F 0 "JP?" H 1350 4785 50  0000 C CNN
+F 1 "Backfeed" H 1350 4694 50  0000 C CNN
+F 2 "OHMC2022:SolderJumper-2_P1.3mm_Open_RoundedPad1.0x1.5mm" H 1350 4600 50  0001 C CNN
+F 3 "~" H 1350 4600 50  0001 C CNN
+	1    1350 4600
+	0    -1   -1   0
+$EndComp
+Wire Wire Line
+	1350 4700 1350 4800
+Wire Wire Line
+	1350 4800 1550 4800
+Wire Wire Line
+	1550 4800 1550 4600
+Wire Wire Line
+	1250 4150 1350 4150
+Wire Wire Line
+	1350 4150 1350 4500
+$Comp
+L power:+3V3 #PWR?
+U 1 1 6142215D
+P 650 4000
+AR Path="/6123BB15/6142215D" Ref="#PWR?"  Part="1"
+AR Path="/611E335F/6142215D" Ref="#PWR?"  Part="1"
+F 0 "#PWR?" H 650 3850 50  0001 C CNN
+F 1 "+3V3" H 665 4173 50  0000 C CNN
+F 2 "" H 650 4000 50  0001 C CNN
+F 3 "" H 650 4000 50  0001 C CNN
+	1    650  4000
+	1    0    0    -1
+$EndComp
+Text Notes 1000 5000 0    50   ~ 0
+Don't do this.\n(Do it. Do IT!)
 $EndSCHEMATC

Commit message: Adding in extra decoupling.
Parts:
- gave numbers to parts that had none: 1
Changed lines of the file:
@@
 	650  4150 950  4150
 $Comp
-L pkl_power:VIN #PWR?
+L pkl_power:VIN #PWR0142
 U 1 1 61405D3E
 P 1550 4600
-F 0 "#PWR?" H 1550 4450 50  0001 C CNN
+F 0 "#PWR0142" H 1550 4450 50  0001 C CNN
 F 1 "VIN" H 1550 4750 50  0000 C CNN
 F 2 "" H 1550 4600 50  0001 C CNN
@@
 P 1350 4600
 AR Path="/6141A32E" Ref="JP?"  Part="1"
-AR Path="/611E335F/6141A32E" Ref="JP?"  Part="1"
-F 0 "JP?" H 1350 4785 50  0000 C CNN
+AR Path="/611E335F/6141A32E" Ref="JP302"  Part="1"
+F 0 "JP302" H 1350 4785 50  0000 C CNN
 F 1 "Backfeed" H 1350 4694 50  0000 C CNN
 F 2 "OHMC2022:SolderJumper-2_P1.3mm_Open_RoundedPad1.0x1.5mm" H 1350 4600 50  0001 C CNN
@@
 P 650 4000
 AR Path="/6123BB15/6142215D" Ref="#PWR?"  Part="1"
-AR Path="/611E335F/6142215D" Ref="#PWR?"  Part="1"
-F 0 "#PWR?" H 650 3850 50  0001 C CNN
+AR Path="/611E335F/6142215D" Ref="#PWR0183"  Part="1"
+F 0 "#PWR0183" H 650 3850 50  0001 C CNN
 F 1 "+3V3" H 665 4173 50  0000 C CNN
 F 2 "" H 650 4000 50  0001 C CNN

Commit message: Trying to add suppliers in Altium formats.
Parts:
- C601, C609, C610: Supplier 1 (none) -> Digi-Key; Supplier Part Number 1 (none) -> 490-3896-1-ND
- C602, C604, C605, C607: Supplier 1 (none) -> Digi-Key; Supplier Part Number 1 (none) -> 587-3352-1-ND
- C603: Supplier 1 (none) -> Digi-Key; Supplier Part Number 1 (none) -> 399-6856-1-ND
- D601, D602: Supplier 1 (none) -> Digi-Key; Supplier Part Number 1 (none) -> RB496EACT-ND
- L601, L602: Supplier 1 (none) -> Digi-Key; Supplier Part Number 1 (none) -> SRN4018-4R7MCT-ND
- R601, R604, R605, R606: Supplier 1 (none) -> Digi-Key; Supplier Part Number 1 (none) -> RHM100KDCT-ND
- R603: Supplier 1 (none) -> Digi-Key; Supplier Part Number 1 (none) -> 311-120KGRCT-ND
- R608, R609: Supplier 1 (none) -> Digi-Key; Supplier Part Number 1 (none) -> 311-0.0GRCT-ND
- R610: Supplier 1 (none) -> Digi-Key; Supplier Part Number 1 (none) -> CR0603-JW-105ELFCT-ND
- R612: Supplier 1 (none) -> Digi-Key; Supplier Part Number 1 (none) -> 311-536KHRCT-ND
- U601: Supplier 1 (none) -> Digi-Key; Supplier Part Number 1 (none) -> PAM2306AYPAADICT-ND
- U602: Supplier 1 (none) -> Digi-Key; Supplier Part Number 1 (none) -> MIC5317-2.5YM5-CT-ND
- U603: Supplier 1 (none) -> Digi-Key; Supplier Part Number 1 (none) -> SIP32431DR3-T1GE3CT-ND
Changed lines of the file:
@@
 F 4 "PAM2306AYPAA" H 4200 3750 50  0001 C CNN "MPN"
 F 5 "PAM2306AYPAADICT-ND" H 4200 3750 50  0001 C CNN "DPN"
+F 6 "Digi-Key" H 4200 3750 50  0001 C CNN "Supplier 1"
+F 7 "PAM2306AYPAADICT-ND" H 4200 3750 50  0001 C CNN "Supplier Part Number 1"
 	1    4200 3750
 	1    0    0    -1
@@
 F 6 "6.3V" H 6465 3655 50  0000 L CNN "Tol"
 F 7 "0603" H 6465 3564 50  0000 L CNN "Pkg"
+F 8 "Digi-Key" H 6350 3700 50  0001 C CNN "Supplier 1"
+F 9 "490-3896-1-ND" H 6350 3700 50  0001 C CNN "Supplier Part Number 1"
 	1    6350 3700
 	1    0    0    -1
@@
 F 6 "6.3V" H 8065 1455 50  0000 L CNN "Tol"
 F 7 "0603" H 8065 1364 50  0000 L CNN "Pkg"
+F 8 "Digi-Key" H 7950 1500 50  0001 C CNN "Supplier 1"
+F 9 "490-3896-1-ND" H 7950 1500 50  0001 C CNN "Supplier Part Number 1"
 	1    7950 1500
 	1    0    0    -1
@@
 F 5 "ESR03EZPJ104" H 5750 4550 50  0001 C CNN "MPN"
 F 6 "RHM100KDCT-ND" H 5750 4550 50  0001 C CNN "DPN"
+F 7 "Digi-Key" H 5750 4550 50  0001 C CNN "Supplier 1"
+F 8 "RHM100KDCT-ND" H 5750 4550 50  0001 C CNN "Supplier Part Number 1"
 	1    5750 4550
 	1    0    0    -1
@@
 F 5 "ESR03EZPJ104" H 5750 4050 50  0001 C CNN "MPN"
 F 6 "RHM100KDCT-ND" H 5750 4050 50  0001 C CNN "DPN"
+F 7 "Digi-Key" H 5750 4050 50  0001 C CNN "Supplier 1"
+F 8 "RHM100KDCT-ND" H 5750 4050 50  0001 C CNN "Supplier Part Number 1"
 	1    5750 4050
 	1    0    0    -1
@@
 F 5 "RC0603JR-07120KL" H 5300 4550 50  0001 C CNN "MPN"
 F 6 "311-120KGRCT-ND" H 5300 4550 50  0001 C CNN "DPN"
+F 7 "Digi-Key" H 5300 4550 50  0001 C CNN "Supplier 1"
+F 8 "311-120KGRCT-ND" H 5300 4550 50  0001 C CNN "Supplier Part Number 1"
 	1    5300 4550
 	1    0    0    -1
@@
 F 4 "SRN4018-4R7M" V 5050 3850 50  0001 C CNN "MPN"
 F 5 "SRN4018-4R7MCT-ND" V 5050 3850 50  0001 C CNN "DPN"
+F 6 "Digi-Key" H 5050 3850 50  0001 C CNN "Supplier 1"
+F 7 "SRN4018-4R7MCT-ND" H 5050 3850 50  0001 C CNN "Supplier Part Number 1"
 	1    5050 3850
 	0    -1   -1   0
@@
 F 4 "SRN4018-4R7M" V 5050 3550 50  0001 C CNN "MPN"
 F 5 "SRN4018-4R7MCT-ND" V 5050 3550 50  0001 C CNN "DPN"
+F 6 "Digi-Key" H 5050 3550 50  0001 C CNN "Supplier 1"
+F 7 "SRN4018-4R7MCT-ND" H 5050 3550 50  0001 C CNN "Supplier Part Number 1"
 	1    5050 3550
 	0    -1   -1   0
@@
 F 6 "6.3V" H 2715 4255 50  0000 L CNN "Tol"
 F 7 "0603" H 2715 4164 50  0000 L CNN "Pkg"
+F 8 "Digi-Key" H 2600 4300 50  0001 C CNN "Supplier 1"
+F 9 "490-3896-1-ND" H 2600 4300 50  0001 C CNN "Supplier Part Number 1"
 	1    2600 4300
 	1    0    0    1
@@
 F 5 "RC0603JR-070RL" H 1450 3550 50  0001 C CNN "MPN"
 F 6 "311-0.0GRCT-ND" H 1450 3550 50  0001 C CNN "DPN"
+F 7 "Digi-Key" H 1450 3550 50  0001 C CNN "Supplier 1"
+F 8 "311-0.0GRCT-ND" H 1450 3550 50  0001 C CNN "Supplier Part Number 1"
 	1    1450 3550
 	0    1    1    0
@@
 F 7 "0603" H 2015 4209 50  0000 L CNN "Pkg"
 F 8 "X7R" H 2015 4118 50  0000 L CNN "TCoff"
+F 9 "Digi-Key" H 1900 4300 50  0001 C CNN "Supplier 1"
+F 10 "587-3352-1-ND" H 1900 4300 50  0001 C CNN "Supplier Part Number 1"
 	1    1900 4300
 	1    0    0    -1
@@
 F 5 "RC0603JR-070RL" H 1450 3850 50  0001 C CNN "MPN"
 F 6 "311-0.0GRCT-ND" H 1450 3850 50  0001 C CNN "DPN"
+F 7 "Digi-Key" H 1450 3850 50  0001 C CNN "Supplier 1"
+F 8 "311-0.0GRCT-ND" H 1450 3850 50  0001 C CNN "Supplier Part Number 1"
 	1    1450 3850
 	0    1    1    0
@@
 F 4 "RB496EATR" H 2350 3700 50  0001 C CNN "MPN"
 F 5 "RB496EACT-ND" H 2350 3700 50  0001 C CNN "DPN"
+F 6 "Digi-Key" H 2350 3700 50  0001 C CNN "Supplier 1"
+F 7 "RB496EACT-ND" H 2350 3700 50  0001 C CNN "Supplier Part Number 1"
 	1    2350 3700
 	1    0    0    -1
@@
 F 4 "RB496EATR" H 1100 4000 50  0001 C CNN "MPN"
 F 5 "RB496EACT-ND" H 1100 4000 50  0001 C CNN "DPN"
+F 6 "Digi-Key" H 1100 4000 50  0001 C CNN "Supplier 1"
+F 7 "RB496EACT-ND" H 1100 4000 50  0001 C CNN "Supplier Part Number 1"
 	1    1100 4000
 	1    0    0    -1
@@
 F 7 "0603" H 9415 3909 50  0000 L CNN "Pkg"
 F 8 "X7R" H 9415 3818 50  0000 L CNN "TCoff"
+F 9 "Digi-Key" H 9300 4000 50  0001 C CNN "Supplier 1"
+F 10 "399-6856-1-ND" H 9300 4000 50  0001 C CNN "Supplier Part Number 1"
 	1    9300 4000
 	1    0    0    -1
@@
 F 7 "0603" H 9915 3909 50  0000 L CNN "Pkg"
 F 8 "X7R" H 9915 3818 50  0000 L CNN "TCoff"
+F 9 "Digi-Key" H 9800 4000 50  0001 C CNN "Supplier 1"
+F 10 "587-3352-1-ND" H 9800 4000 50  0001 C CNN "Supplier Part Number 1"
 	1    9800 4000
 	1    0    0    -1
@@
 F 7 "0603" H 8165 3959 50  0000 L CNN "Pkg"
 F 8 "X7R" H 8165 3868 50  0000 L CNN "TCoff"
+F 9 "Digi-Key" H 8050 4050 50  0001 C CNN "Supplier 1"
+F 10 "587-3352-1-ND" H 8050 4050 50  0001 C CNN "Supplier Part Number 1"
 	1    8050 4050
 	1    0    0    -1
@@
 F 4 "MIC5317-2.5YM5-TR" H 8800 3900 50  0001 C CNN "MPN"
 F 5 "MIC5317-2.5YM5-CT-ND" H 8800 3900 50  0001 C CNN "DPN"
+F 6 "Digi-Key" H 8800 3900 50  0001 C CNN "Supplier 1"
+F 7 "MIC5317-2.5YM5-CT-ND" H 8800 3900 50  0001 C CNN "Supplier Part Number 1"
 	1    8800 3900
 	1    0    0    -1
@@
 F 5 "ESR03EZPJ104" H 5800 1650 50  0001 C CNN "MPN"
 F 6 "RHM100KDCT-ND" H 5800 1650 50  0001 C CNN "DPN"
+F 7 "Digi-Key" H 5800 1650 50  0001 C CNN "Supplier 1"
+F 8 "RHM100KDCT-ND" H 5800 1650 50  0001 C CNN "Supplier Part Number 1"
 	1    5800 1650
 	1    0    0    -1
@@
 F 4 "SIP32431DR3-T1GE3" H 7100 1900 50  0001 C CNN "MPN"
 F 5 "SIP32431DR3-T1GE3CT-ND" H 7100 1900 50  0001 C CNN "DPN"
+F 6 "Digi-Key" H 7100 1900 50  0001 C CNN "Supplier 1"
+F 7 "SIP32431DR3-T1GE3CT-ND" H 7100 1900 50  0001 C CNN "Supplier Part Number 1"
 	1    7100 1900
 	1    0    0    -1
@@
 F 7 "0603" H 5915 2159 50  0000 L CNN "Pkg"
 F 8 "X7R" H 5915 2068 50  0000 L CNN "TCoff"
+F 9 "Digi-Key" H 5800 2250 50  0001 C CNN "Supplier 1"
+F 10 "587-3352-1-ND" H 5800 2250 50  0001 C CNN "Supplier Part Number 1"
 	1    5800 2250
 	1    0    0    -1
@@
 F 5 "CR0603-JW-105ELF" H 6350 2300 50  0001 C CNN "MPN"
 F 6 "CR0603-JW-105ELFCT-ND" H 6350 2300 50  0001 C CNN "DPN"
+F 7 "Digi-Key" H 6350 2300 50  0001 C CNN "Supplier 1"
+F 8 "CR0603-JW-105ELFCT-ND" H 6350 2300 50  0001 C CNN "Supplier Part Number 1"
 	1    6350 2300
 	1    0    0    -1
@@
 F 5 "RC0603FR-07536KL" H 5300 4050 50  0001 C CNN "MPN"
 F 6 "311-536KHRCT-ND" H 5300 4050 50  0001 C CNN "DPN"
+F 7 "Digi-Key" H 5300 4050 50  0001 C CNN "Supplier 1"
+F 8 "311-536KHRCT-ND" H 5300 4050 50  0001 C CNN "Supplier Part Number 1"
 	1    5300 4050
 	1    0    0    -1
@@
 F 5 "ESR03EZPJ104" H 3650 4300 50  0001 C CNN "MPN"
 F 6 "RHM100KDCT-ND" H 3650 4300 50  0001 C CNN "DPN"
+F 7 "Digi-Key" H 3650 4300 50  0001 C CNN "Supplier 1"
+F 8 "RHM100KDCT-ND" H 3650 4300 50  0001 C CNN "Supplier Part Number 1"
 	1    3650 4300
 	1    0    0    -1
