File: Hardware/Power.sch (KiCad schematic (older format))
At the start: 25 parts, among them U601 PAM2306AYPAA, U602 MIC5317-2.5YM5, U603 SiP32431DR3

Commit message: Routing.
Parts:
- added C303, C306, C310: 0.1uF, Capacitor_SMD:C_0603_1608Metric, symbol Device:C
- added R302: 0R, Resistor_SMD:R_0603_1608Metric, symbol Device:R_Small
Connections:
- net +1V2: now also C310.1
- net +5V: now also C303.1
- net GND: now also C303.2, C306.2, C310.2
- net at C601.2, U601.6 (EN1), U601.7 (VIN1): now also R302.1; no longer D601.4 (K2), D601.5 (K1)
- new net: C306.1, D601.4 (K2), D601.5 (K1), R302.2
Other:
- moved on the sheet: C601
Changed lines of the file:
@@
 Wire Wire Line
 	3650 3650 3650 3550
-Connection ~ 3650 3550
 Wire Wire Line
 	3800 3850 3650 3850
@@
 Wire Wire Line
 	2600 3850 2600 3550
-Connection ~ 2600 3550
 $Comp
 L Device:C C601
 U 1 1 613F36D2
-P 2600 4300
-F 0 "C601" H 2715 4437 50  0000 L CNN
-F 1 "10uF" H 2715 4346 50  0000 L CNN
-F 2 "Capacitor_SMD:C_0603_1608Metric" H 2638 4150 50  0001 C CNN
-F 3 "~" H 2600 4300 50  0001 C CNN
-F 4 "GRM188R60J106ME47D" H 2600 4300 50  0001 C CNN "MPN"
-F 5 "490-3896-1-ND" H 2600 4300 50  0001 C CNN "DPN"
-F 6 "6.3V" H 2715 4255 50  0000 L CNN "Tol"
-F 7 "0603" H 2715 4164 50  0000 L CNN "Pkg"
-F 8 "Digi-Key" H 2600 4300 50  0001 C CNN "Supplier 1"
-F 9 "490-3896-1-ND" H 2600 4300 50  0001 C CNN "Supplier Part Number 1"
-	1    2600 4300
+P 3150 4300
+F 0 "C601" H 3265 4437 50  0000 L CNN
+F 1 "10uF" H 3265 4346 50  0000 L CNN
+F 2 "Capacitor_SMD:C_0603_1608Metric" H 3188 4150 50  0001 C CNN
+F 3 "~" H 3150 4300 50  0001 C CNN
+F 4 "GRM188R60J106ME47D" H 3150 4300 50  0001 C CNN "MPN"
+F 5 "490-3896-1-ND" H 3150 4300 50  0001 C CNN "DPN"
+F 6 "6.3V" H 3265 4255 50  0000 L CNN "Tol"
+F 7 "0603" H 3265 4164 50  0000 L CNN "Pkg"
+F 8 "Digi-Key" H 3150 4300 50  0001 C CNN "Supplier 1"
+F 9 "490-3896-1-ND" H 3150 4300 50  0001 C CNN "Supplier Part Number 1"
+	1    3150 4300
 	1    0    0    1
 $EndComp
@@
 	3650 3950 3650 3850
 Wire Wire Line
-	2600 3550 3650 3550
-Wire Wire Line
 	5800 1450 5800 1550
 Wire Wire Line
@@
 Text Notes 1000 5000 0    50   ~ 0
 Don't do this.\n(Do it. Do IT!)
+$Comp
+L Device:C C310
+U 1 1 61476322
+P 6850 3700
+F 0 "C310" H 6965 3882 50  0000 L CNN
+F 1 "0.1uF" H 6965 3791 50  0000 L CNN
+F 2 "Capacitor_SMD:C_0603_1608Metric" H 6888 3550 50  0001 C CNN
+F 3 "~" H 6850 3700 50  0001 C CNN
+F 4 "C0603C104K5RACAUTO" H 6850 3700 50  0001 C CNN "MPN"
+F 5 "399-6856-1-ND" H 6850 3700 50  0001 C CNN "DPN"
+F 6 "50V" H 6965 3700 50  0000 L CNN "Tol"
+F 7 "0603" H 6965 3609 50  0000 L CNN "Pkg"
+F 8 "X7R" H 6965 3518 50  0000 L CNN "TCoff"
+F 9 "Digi-Key" H 6850 3700 50  0001 C CNN "Supplier 1"
+F 10 "399-6856-1-ND" H 6850 3700 50  0001 C CNN "Supplier Part Number 1"
+	1    6850 3700
+	1    0    0    -1
+$EndComp
+$Comp
+L power:+1V2 #PWR?
+U 1 1 61478A71
+P 6850 3500
+AR Path="/6123BB15/61478A71" Ref="#PWR?"  Part="1"
+AR Path="/611E335F/61478A71" Ref="#PWR0304"  Part="1"
+F 0 "#PWR0304" H 6850 3350 50  0001 C CNN
+F 1 "+1V2" H 6865 3673 50  0000 C CNN
+F 2 "" H 6850 3500 50  0001 C CNN
+F 3 "" H 6850 3500 50  0001 C CNN
+	1    6850 3500
+	1    0    0    -1
+$EndComp
+Wire Wire Line
+	6850 3500 6850 3550
+$Comp
+L power:GND #PWR?
+U 1 1 6147B57E
+P 6850 3950
+AR Path="/611E3335/6147B57E" Ref="#PWR?"  Part="1"
+AR Path="/611E335F/6147B57E" Ref="#PWR0305"  Part="1"
+F 0 "#PWR0305" H 6850 3700 50  0001 C CNN
+F 1 "GND" H 6855 3777 50  0000 C CNN
+F 2 "" H 6850 3950 50  0001 C CNN
+F 3 "" H 6850 3950 50  0001 C CNN
+	1    6850 3950
+	-1   0    0    -1
+$EndComp
+Wire Wire Line
+	6850 3950 6850 3850
+$Comp
+L Device:C C303
+U 1 1 61491D89
+P 2250 2450
+F 0 "C303" H 2365 2632 50  0000 L CNN
+F 1 "0.1uF" H 2365 2541 50  0000 L CNN
+F 2 "Capacitor_SMD:C_0603_1608Metric" H 2288 2300 50  0001 C CNN
+F 3 "~" H 2250 2450 50  0001 C CNN
+F 4 "C0603C104K5RACAUTO" H 2250 2450 50  0001 C CNN "MPN"
+F 5 "399-6856-1-ND" H 2250 2450 50  0001 C CNN "DPN"
+F 6 "50V" H 2365 2450 50  0000 L CNN "Tol"
+F 7 "0603" H 2365 2359 50  0000 L CNN "Pkg"
+F 8 "X7R" H 2365 2268 50  0000 L CNN "TCoff"
+F 9 "Digi-Key" H 2250 2450 50  0001 C CNN "Supplier 1"
+F 10 "399-6856-1-ND" H 2250 2450 50  0001 C CNN "Supplier Part Number 1"
+	1    2250 2450
+	1    0    0    -1
+$EndComp
+$Comp
+L power:GND #PWR?
+U 1 1 61491D96
+P 2250 2700
+AR Path="/611E3335/61491D96" Ref="#PWR?"  Part="1"
+AR Path="/611E335F/61491D96" Ref="#PWR0302"  Part="1"
+F 0 "#PWR0302" H 2250 2450 50  0001 C CNN
+F 1 "GND" H 2255 2527 50  0000 C CNN
+F 2 "" H 2250 2700 50  0001 C CNN
+F 3 "" H 2250 2700 50  0001 C CNN
+	1    2250 2700
+	-1   0    0    -1
+$EndComp
+Wire Wire Line
+	2250 2700 2250 2600
+$Comp
+L power:+5V #PWR?
+U 1 1 6149486E
+P 2250 2150
+AR Path="/6123BB15/6149486E" Ref="#PWR?"  Part="1"
+AR Path="/611E335F/6149486E" Ref="#PWR0301"  Part="1"
+F 0 "#PWR0301" H 2250 2000 50  0001 C CNN
+F 1 "+5V" H 2265 2323 50  0000 C CNN
+F 2 "" H 2250 2150 50  0001 C CNN
+F 3 "" H 2250 2150 50  0001 C CNN
+	1    2250 2150
+	1    0    0    -1
+$EndComp
+Wire Wire Line
+	2250 2150 2250 2300
+$Comp
+L Device:C C306
+U 1 1 614AD8E8
+P 2600 4300
+F 0 "C306" H 2715 4482 50  0000 L CNN
+F 1 "0.1uF" H 2715 4391 50  0000 L CNN
+F 2 "Capacitor_SMD:C_0603_1608Metric" H 2638 4150 50  0001 C CNN
+F 3 "~" H 2600 4300 50  0001 C CNN
+F 4 "C0603C104K5RACAUTO" H 2600 4300 50  0001 C CNN "MPN"
+F 5 "399-6856-1-ND" H 2600 4300 50  0001 C CNN "DPN"
+F 6 "50V" H 2715 4300 50  0000 L CNN "Tol"
+F 7 "0603" H 2715 4209 50  0000 L CNN "Pkg"
+F 8 "X7R" H 2715 4118 50  0000 L CNN "TCoff"
+F 9 "Digi-Key" H 2600 4300 50  0001 C CNN "Supplier 1"
+F 10 "399-6856-1-ND" H 2600 4300 50  0001 C CNN "Supplier Part Number 1"
+	1    2600 4300
+	1    0    0    -1
+$EndComp
+Wire Wire Line
+	2600 3550 2750 3550
+Connection ~ 2600 3550
+Wire Wire Line
+	2950 3550 3150 3550
+Wire Wire Line
+	3150 3550 3150 4150
+$Comp
+L power:GND #PWR?
+U 1 1 614C10F8
+P 3150 4800
+AR Path="/611E3335/614C10F8" Ref="#PWR?"  Part="1"
+AR Path="/611E335F/614C10F8" Ref="#PWR0303"  Part="1"
+F 0 "#PWR0303" H 3150 4550 50  0001 C CNN
+F 1 "GND" H 3155 4627 50  0000 C CNN
+F 2 "" H 3150 4800 50  0001 C CNN
+F 3 "" H 3150 4800 50  0001 C CNN
+	1    3150 4800
+	-1   0    0    -1
+$EndComp
+Wire Wire Line
+	3150 4450 3150 4800
+Wire Wire Line
+	3150 3550 3650 3550
+Connection ~ 3150 3550
+Connection ~ 3650 3550
+$Comp
+L Device:R_Small R302
+U 1 1 614C9935
+P 2850 3550
+F 0 "R302" H 2909 3596 50  0000 L CNN
+F 1 "0R" H 2909 3505 50  0000 L CNN
+F 2 "Resistor_SMD:R_0603_1608Metric" V 2780 3550 50  0001 C CNN
+F 3 "~" H 2850 3550 50  0001 C CNN
+F 4 "0603" H 3000 3700 50  0000 C CNN "Pkg"
+F 5 "RC0603JR-070RL" H 2850 3550 50  0001 C CNN "MPN"
+F 6 "311-0.0GRCT-ND" H 2850 3550 50  0001 C CNN "DPN"
+F 7 "Digi-Key" H 2850 3550 50  0001 C CNN "Supplier 1"
+F 8 "311-0.0GRCT-ND" H 2850 3550 50  0001 C CNN "Supplier Part Number 1"
+	1    2850 3550
+	0    1    1    0
+$EndComp
 $EndSCHEMATC

Commit message: Putting down some final touches on layout, initial DRC.
Changed lines of the file:
@@
 	5200 3550 5750 3550
 Wire Wire Line
-	5750 3550 5750 3900
+	5750 3550 5750 3700
 Wire Wire Line
 	5750 4200 5750 4400
@@
 	6350 1450 5800 1450
 Wire Wire Line
-	7550 1300 7550 1800
+	7550 1300 7550 1450
 Wire Wire Line
 	7550 1800 7400 1800
@@
 $EndComp
 Wire Wire Line
-	2250 2150 2250 2300
+	2250 2150 2250 2250
 $Comp
 L Device:C C306
@@
 	0    1    1    0
 $EndComp
+$Comp
+L power:PWR_FLAG #FLG?
+U 1 1 617195E6
+P 1950 2200
+F 0 "#FLG?" H 1950 2275 50  0001 C CNN
+F 1 "PWR_FLAG" H 1950 2373 50  0000 C CNN
+F 2 "" H 1950 2200 50  0001 C CNN
+F 3 "~" H 1950 2200 50  0001 C CNN
+	1    1950 2200
+	1    0    0    -1
+$EndComp
+Wire Wire Line
+	1950 2200 1950 2250
+Wire Wire Line
+	1950 2250 2250 2250
+Connection ~ 2250 2250
+Wire Wire Line
+	2250 2250 2250 2300
+$Comp
+L power:PWR_FLAG #FLG?
+U 1 1 61723033
+P 5500 1400
+F 0 "#FLG?" H 5500 1475 50  0001 C CNN
+F 1 "PWR_FLAG" H 5500 1573 50  0000 C CNN
+F 2 "" H 5500 1400 50  0001 C CNN
+F 3 "~" H 5500 1400 50  0001 C CNN
+	1    5500 1400
+	1    0    0    -1
+$EndComp
+Wire Wire Line
+	5500 1400 5500 1450
+Wire Wire Line
+	5500 1450 5800 1450
+$Comp
+L power:PWR_FLAG #FLG?
+U 1 1 61726C76
+P 7250 1400
+F 0 "#FLG?" H 7250 1475 50  0001 C CNN
+F 1 "PWR_FLAG" H 7250 1573 50  0000 C CNN
+F 2 "" H 7250 1400 50  0001 C CNN
+F 3 "~" H 7250 1400 50  0001 C CNN
+	1    7250 1400
+	1    0    0    -1
+$EndComp
+Wire Wire Line
+	7250 1400 7250 1450
+Wire Wire Line
+	7250 1450 7550 1450
+$Comp
+L power:PWR_FLAG #FLG?
+U 1 1 6172BD15
+P 10100 3750
+F 0 "#FLG?" H 10100 3825 50  0001 C CNN
+F 1 "PWR_FLAG" H 10100 3923 50  0000 C CNN
+F 2 "" H 10100 3750 50  0001 C CNN
+F 3 "~" H 10100 3750 50  0001 C CNN
+	1    10100 3750
+	-1   0    0    -1
+$EndComp
+Wire Wire Line
+	10100 3750 10100 3800
+Wire Wire Line
+	10100 3800 9800 3800
+$Comp
+L power:PWR_FLAG #FLG?
+U 1 1 6172FD09
+P 6050 3650
+F 0 "#FLG?" H 6050 3725 50  0001 C CNN
+F 1 "PWR_FLAG" H 6050 3823 50  0000 C CNN
+F 2 "" H 6050 3650 50  0001 C CNN
+F 3 "~" H 6050 3650 50  0001 C CNN
+	1    6050 3650
+	-1   0    0    -1
+$EndComp
+Wire Wire Line
+	6050 3650 6050 3700
+Wire Wire Line
+	6050 3700 5750 3700
+Connection ~ 5750 3700
+Wire Wire Line
+	5750 3700 5750 3900
+Connection ~ 7550 1450
+Wire Wire Line
+	7550 1450 7550 1800
 $EndSCHEMATC

Commit message: Cleaning up some libraries, better if those pins are connected.
Changed lines of the file:
@@
 Wire Wire Line
 	7550 1450 7550 1800
+$Comp
+L power:PWR_FLAG #FLG?
+U 1 1 617ED9CA
+P 3150 3450
+AR Path="/617ED9CA" Ref="#FLG?"  Part="1"
+AR Path="/611E335F/617ED9CA" Ref="#FLG0107"  Part="1"
+F 0 "#FLG0107" H 3150 3525 50  0001 C CNN
+F 1 "PWR_FLAG" H 3150 3623 50  0000 C CNN
+F 2 "" H 3150 3450 50  0001 C CNN
+F 3 "~" H 3150 3450 50  0001 C CNN
+	1    3150 3450
+	1    0    0    -1
+$EndComp
+Wire Wire Line
+	3150 3450 3150 3550
 $EndSCHEMATC

Commit message: And just cleaning up the power flags a little.
Changed lines of the file:
@@
-$Comp
-L power:PWR_FLAG #FLG?
-U 1 1 6172BD15
-P 10100 3750
-AR Path="/6172BD15" Ref="#FLG?"  Part="1"
-AR Path="/611E335F/6172BD15" Ref="#FLG0105"  Part="1"
-F 0 "#FLG0105" H 10100 3825 50  0001 C CNN
-F 1 "PWR_FLAG" H 10100 3923 50  0000 C CNN
-F 2 "" H 10100 3750 50  0001 C CNN
-F 3 "~" H 10100 3750 50  0001 C CNN
-	1    10100 3750
-	-1   0    0    -1
-$EndComp
-Wire Wire Line
-	10100 3750 10100 3800
-Wire Wire Line
-	10100 3800 9800 3800
 $Comp
 L power:PWR_FLAG #FLG?
